Commit message: adding mesh file for camera

File: src/slam/urdf/prototype.urdf.xacro (robot description, xacro)
@@ -122,5 +122,5 @@
 			<origin rpy="0 0 0" xyz="0 0 0"/>
 			<geometry>
-					<box size="${lk} ${bk} ${hk}"/>
+					<mesh filename="package://mybot_description/meshes/kinect.dae"/>
 			</geometry>
 		</visual>
